File: hardware/twinkle-led-controller.sch (KiCad schematic (older format))
At the start: 25 parts, among them J1 USB_B_Micro, J2 Conn_01x05, Q1 Q_NPN_BEC, Q2 Q_NPN_BEC, SW1 SW_Push, U1 AZ1117-3.3, U2 INTERFACE-CP2102-GMR(QFN28), U3 ESP32-WROOM-32

Commit message: Hardware revision 1.1:
- Fix pins to not use flash pins
- Fix screw terminal footprint (holes were too small)
- Add screw terminal for power
- Add out for multi-unit synchronization
Parts:
- added J12: Screw_Terminal_01x02, homebrew:Wurth_ScrewTerminal_1x02_P5.00mm_691137710002, symbol Connector:Screw_Terminal_01x02
- U2: symbol snapeda-CP2102:INTERFACE-CP2102-GMR(QFN28) -> twinkle-led-controller-rescue:INTERFACE-CP2102-GMR(QFN28)-snapeda-CP2102
Connections:
- net LED9_A is gone; now on net LED8_A: U3.8 (IO32)
- net LED9_B is gone; now on net LED8_B: U3.9 (IO33)
- net +5V: now also J12.1 (Pin_1)
- net GND: now also J12.2 (Pin_2)
- net LED2_A: now also U3.29 (IO5); no longer U3.28 (IO17)
- net LED3_A: now also U3.27 (IO16); no longer U3.26 (IO4)
- net LED3_B: now also U3.28 (IO17); no longer U3.27 (IO16)
- net LED4_A: now also U3.24 (IO2); no longer U3.21 (SDO/SD0)
- net LED4_B: now also U3.26 (IO4); no longer U3.22 (SDI/SD1)
- net LED5_A: now also U3.16 (IO13); no longer U3.18 (SWP/SD3)
- net LED5_B: now also U3.23 (IO15); no longer U3.20 (SCK/CLK)
- net LED6_A: now also U3.12 (IO27); no longer U3.16 (IO13)
- net LED6_B: now also U3.13 (IO14); no longer U3.17 (SHD/SD2)
- net LED7_A: now also U3.10 (IO25); no longer U3.12 (IO27)
- net LED7_B: now also U3.11 (IO26); no longer U3.13 (IO14)
- net LED8_A: no longer U3.10 (IO25)
- net LED8_B: no longer U3.11 (IO26)
- net AUX_OUT: now reaches U3.14 (IO12)
- net AUX_OUT: now also D2.2 (A), J2.3 (Pin_3)
- net AUX0 renamed AUX_IN
- net AUX1: no longer names the net of U3.5 (SENSOR_VN)
- net AUX1: no longer J2.3 (Pin_3)
- net LED_BUILTIN: no longer names the net of U3.19 (SCS/CMD)
- net LED_BUILTIN: no longer D2.2 (A)
- no-connect marks 25 -> 28
Changed lines of the file:
@@
 $Descr A4 11693 8268
 encoding utf-8
-Sheet 1 11
+Sheet 1 10
 Title ""
 Date ""
@@
 	1    0    0    -1
 $EndComp
-NoConn ~ 5600 2300
-NoConn ~ 5600 2000
-NoConn ~ 5600 1600
-NoConn ~ 5600 1900
 Text Label 5650 2900 0    50   ~ 0
 LED0_A
@@
 	5650 2400 5600 2400
 Text Label 5650 2500 0    50   ~ 0
-LED2_A
+LED3_B
 Wire Wire Line
 	5650 2500 5600 2500
@@
 	5650 2600 5600 2600
 Text Label 5650 1800 0    50   ~ 0
-LED3_A
+LED4_B
 Wire Wire Line
 	5650 2700 5600 2700
 Text Label 5650 2400 0    50   ~ 0
-LED3_B
+LED3_A
 Wire Wire Line
 	5650 2800 5600 2800
 Wire Wire Line
 	5650 2900 5600 2900
-Text Label 4350 2700 2    50   ~ 0
-LED4_B
+Text Label 5650 1900 0    50   ~ 0
+LED2_A
 Wire Wire Line
 	5650 3000 5600 3000
-Text Label 4350 2900 2    50   ~ 0
-LED5_A
 Wire Wire Line
 	5650 3100 5600 3100
-Text Label 4350 3000 2    50   ~ 0
-LED5_B
 Wire Wire Line
 	5650 3200 5600 3200
 Text Label 5650 2100 0    50   ~ 0
-LED6_A
+LED5_A
 Wire Wire Line
 	5650 3300 5600 3300
-Text Label 4350 2800 2    50   ~ 0
-LED6_B
+Text Label 5650 2300 0    50   ~ 0
+LED5_B
 Wire Wire Line
 	5650 3400 5600 3400
 Text Label 5650 3300 0    50   ~ 0
-LED7_A
+LED6_A
 Wire Wire Line
 	5650 3500 5600 3500
 Text Label 5650 2200 0    50   ~ 0
+LED6_B
+Text Label 5650 3100 0    50   ~ 0
+LED7_A
+Text Label 5650 3200 0    50   ~ 0
 LED7_B
-Text Label 5650 3100 0    50   ~ 0
-LED8_A
-Text Label 5650 3200 0    50   ~ 0
-LED8_B
 Wire Wire Line
 	4350 2600 4400 2600
 Text Label 5650 3400 0    50   ~ 0
-LED9_A
+LED8_A
 Wire Wire Line
 	4350 2700 4400 2700
 Text Label 5650 3500 0    50   ~ 0
-LED9_B
+LED8_B
 Wire Wire Line
 	4350 2800 4400 2800
-Text Label 4350 3100 2    50   ~ 0
-LED_BUILTIN
+Text Label 5650 2000 0    50   ~ 0
+AUX_OUT
 Wire Wire Line
 	4350 3100 4400 3100
@@
 $EndComp
 Text Label 3800 4400 2    50   ~ 0
-LED_BUILTIN
+AUX_OUT
 $Comp
 L power:GND #PWR015
@@
 	3800 4800 3800 4700
 Text Label 4350 1600 2    50   ~ 0
-AUX0
+AUX_IN
 Wire Wire Line
 	4350 1600 4400 1600
-Text Label 4350 1700 2    50   ~ 0
-AUX1
-Wire Wire Line
-	4350 1700 4400 1700
 $Comp
 L Connector_Generic:Conn_01x05 J2
@@
 $EndComp
 Text Label 4000 6050 0    50   ~ 0
-AUX0
+AUX_IN
 Text Label 4000 5950 0    50   ~ 0
-AUX1
+AUX_OUT
 $Comp
 L power:+5V #PWR019
@@
 Wire Wire Line
 	9000 3750 9100 3750
-Text Label 9000 4600 2    50   ~ 0
-LED9_B
-Text Label 9000 4400 2    50   ~ 0
-LED9_A
-$Sheet
-S 9100 4250 550  500
-U 5F6A41C2
-F0 "sheet5F6A41C2" 50
-F1 "LED-output.sch" 50
-F2 "LED_A" I L 9100 4400 50
-F3 "LED_B" I L 9100 4600 50
-$EndSheet
-Wire Wire Line
-	9000 4400 9100 4400
-Wire Wire Line
-	9000 4600 9100 4600
-Text Label 4350 2600 2    50   ~ 0
-LED4_A
 $Comp
 L Device:R R14
@@
 $EndComp
 $Comp
-L snapeda-CP2102:INTERFACE-CP2102-GMR(QFN28) U2
+L twinkle-led-controller-rescue:INTERFACE-CP2102-GMR(QFN28)-snapeda-CP2102 U2
 U 1 1 5F4A17F8
 P 2250 3900
@@
 NoConn ~ 2050 3100
 NoConn ~ 2450 3700
+NoConn ~ 4350 3100
+NoConn ~ 4350 3000
+NoConn ~ 4350 2900
+NoConn ~ 4350 2800
+NoConn ~ 4350 2700
+NoConn ~ 4350 2600
+Wire Wire Line
+	5650 1600 5600 1600
+Wire Wire Line
+	5650 1900 5600 1900
+Wire Wire Line
+	5650 2300 5600 2300
+Wire Wire Line
+	5600 2000 5650 2000
+Text Label 5650 1600 0    50   ~ 0
+LED4_A
+$Comp
+L Connector:Screw_Terminal_01x02 J12
+U 1 1 5F629BB0
+P 2450 850
+F 0 "J12" H 2530 842 50  0000 L CNN
+F 1 "Screw_Terminal_01x02" H 2530 751 50  0000 L CNN
+F 2 "homebrew:Wurth_ScrewTerminal_1x02_P5.00mm_691137710002" H 2450 850 50  0001 C CNN
+F 3 "~" H 2450 850 50  0001 C CNN
+	1    2450 850
+	1    0    0    -1
+$EndComp
+Wire Wire Line
+	2250 850  1750 850
+Connection ~ 1750 850
+Wire Wire Line
+	1750 1150 2200 1150
+Wire Wire Line
+	2200 1150 2200 950
+Wire Wire Line
+	2200 950  2250 950
+Connection ~ 1750 1150
+NoConn ~ 4400 1700
 $EndSCHEMATC
